Commit message: Add files via upload

File: gewu/Project/Assets/RL-Playground/urdf/zq_humanoid/zq_sa01.urdf (robot description, URDF)
Before this commit: robot zqsa01, 13 links, 12 joints
Links:
- link leg_l6_link: geometry collision box size=0.24 0.08 0.03; visual mesh filename=package://meshes/LeftLeg_Link_06.STL
- link leg_r6_link: geometry collision box size=0.24 0.08 0.03; visual mesh filename=package://meshes/RightLeg_Link_06.STL
