Commit message: gewu 3.0

File: gewu/Assets/urdf/azureLoong_description/AzureLoong.urdf (robot description, URDF)
Before this commit: robot OpenLoog, 32 links, 31 joints
Links:
- link Link_head_pitch: geometry collision mesh filename=package://meshes/Link_head_pitch.STL; visual mesh filename=package://meshes/Link_head_pitch.STL
- link Link_head_yaw: geometry collision mesh filename=package://meshes/Link_head_yaw.STL; visual mesh filename=package://meshes/Link_head_yaw.STL
