Commit message: gewu 3.0

File: gewu/Assets/course/ur5_robotiq/robotiq_85.urdf (robot description, URDF)
Before this commit: robot robotiq_arg2f_85_model, 11 links, 10 joints
Links:
- link left_inner_finger: geometry collision mesh filename=package://meshes/robotiq_85/collision/robotiq_arg2f_85_inne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 scale=0.001 0.001 0.001; visual mesh filename=package://meshes/robotiq_85/visual/robotiq_arg2f_85_inner_f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 scale=0.001 0.001 0.001
- link left_inner_knuckle: geometry collision mesh filename=package://meshes/robotiq_85/collision/robotiq_arg2f_85_inne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 scale=0.001 0.001 0.001; visual mesh filename=package://meshes/robotiq_85/visual/robotiq_arg2f_85_inner_k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 scale=0.001 0.001 0.001
- link left_outer_finger: geometry collision mesh filename=package://meshes/robotiq_85/collision/robotiq_arg2f_85_oute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 scale=0.001 0.001 0.001; visual mesh filename=package://meshes/robotiq_85/visual/robotiq_arg2f_85_outer_f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 scale=0.001 0.001 0.001
- link left_outer_knuckle: geometry collision mesh filename=package://meshes/robotiq_85/collision/robotiq_arg2f_85_oute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 scale=0.001 0.001 0.001; visual mesh filename=package://meshes/robotiq_85/visual/robotiq_arg2f_85_outer_k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 scale=0.001 0.001 0.001
- link right_inner_finger: geometry collision mesh filename=package://meshes/robotiq_85/collision/robotiq_arg2f_85_inne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 scale=0.001 0.001 0.001; visual mesh filename=package://meshes/robotiq_85/visual/robotiq_arg2f_85_inner_f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 scale=0.001 0.001 0.001
- link right_inner_knuckle: geometry collision mesh filename=package://meshes/robotiq_85/collision/robotiq_arg2f_85_inne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 scale=0.001 0.001 0.001; visual mesh filename=package://meshes/robotiq_85/visual/robotiq_arg2f_85_inner_k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 scale=0.001 0.001 0.001
- link right_outer_finger: geometry collision mesh filename=package://meshes/robotiq_85/collision/robotiq_arg2f_85_oute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 scale=0.001 0.001 0.001; visual mesh filename=package://meshes/robotiq_85/visual/robotiq_arg2f_85_outer_f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 scale=0.001 0.001 0.001
- link right_outer_knuckle: geometry collision mesh filename=package://meshes/robotiq_85/collision/robotiq_arg2f_85_oute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 scale=0.001 0.001 0.001; visual mesh filename=package://meshes/robotiq_85/visual/robotiq_arg2f_85_outer_k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 scale=0.001 0.001 0.001
- link robotiq_arg2f_base_link: geometry collision mesh filename=package://meshes/robotiq_85/collision/robotiq_arg2f_base_li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; visual mesh filename=package://meshes/robotiq_85/visual/robotiq_arg2f_85_base_li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 scale=0.001 0.001 0.001
